File: pipes/pipes_outputs.kicad_sch (KiCad schematic)
At the start: 80 parts, among them J10 3.5mm Jack, J11 3.5mm Jack, J12 3.5mm Jack, J5 3.5mm Jack, J6 3.5mm Jack, J7 3.5mm Jack, J8 3.5mm Jack, J9 3.5mm Jack, U20 VTL5C, U21 VTL5C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

Commit message: Adds harmonic outputs
Parts:
- R50, R51, R52, R59, R60, R61, R66, R67: value 43K -> 24.9K; LCSC Part # C17695 -> C137761
Connections:
- net F1 renamed Clk
Other:
- note added: "~30K on"
- moved on the sheet: C54, C55, C56, C57, C58, C59, C60, C61, C62, C63, C64, C65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
