File: pipes_main/pipes_parts.kicad_sch (KiCad schematic)
At the start: 28 parts, among them J3 Eurorack Power Cable

Commit message: Swaps bamboo silkscreen for face logo.
Parts:
- GR2: footprint panel:bamboo_big_neg -> panel:face_logo
Changed lines of the file:
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@@
     (property "Reference" "GR2" (id 0) (at 158.75 73.6305 0))
     (property "Value" "bamboo" (id 1) (at 158.75 76.4056 0))
-    (property "Footprint" "panel:bamboo_big_neg" (id 2) (at 158.75 78.74 0)
+    (property "Footprint" "panel:face_logo" (id 2) (at 158.75 78.74 0)
       (effects (font (size 1.27 1.27)) hide)
     )

Commit message: Adds digikey bom merge. Uses local graphics for panel.
Adds bambooh graphics
Parts:
- KN1: Digi-Key Part 1722-1241-ND -> 1722-1238-ND
Changed lines of the file:
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@@
       (effects (font (size 1.27 1.27)) hide)
     )
-    (property "Digi-Key Part" "1722-1241-ND" (id 4) (at 127 71.755 0)
+    (property "Digi-Key Part" "1722-1238-ND" (id 4) (at 127 71.755 0)
       (effects (font (size 1.27 1.27)) hide)
     )
